File: hardware/led_controller/led_controller.sch (KiCad schematic (older format))
At the start: 38 parts, among them J1 Barrel_Jack_Switch, J2 Conn_01x06, J3 Conn_01x04, J4 Screw_Terminal_01x04, Q1 BC807, Q2 IRLML0030TRPBF-1, Q3 BC807, Q4 IRLML0030TRPBF-1, Q5 BC807, Q6 IRLML0030TRPBF-1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

Commit message: Removed bakers clamps. reduced board size to 55x50 mm
Parts:
- removed D1, D2, D3: 1N4148W, Diode_SMD:D_SOD-123, symbol Diode:1N4148W
- removed JP1: Red, Jumper:SolderJumper-2_P1.3mm_Open_RoundedPad1.0x1.5mm, symbol Jumper:SolderJumper_2_Open
- removed JP2: Green, Jumper:SolderJumper-2_P1.3mm_Open_RoundedPad1.0x1.5mm, symbol Jumper:SolderJumper_2_Open
- removed JP3: Blue, Jumper:SolderJumper-2_P1.3mm_Open_RoundedPad1.0x1.5mm, symbol Jumper:SolderJumper_2_Open
- added R12: 100K, Resistor_SMD:R_0805_2012Metric_Pad1.15x1.40mm_HandSolder, symbol Device:R_Small
Connections:
- net +12V: now also J3.4 (Pin_4), J4.4 (Pin_4), R12.2; no longer J3.1 (Pin_1), J4.1 (Pin_1)
- net DRAIN_BLUE: now also J3.3 (Pin_3), J4.3 (Pin_3); no longer J3.4 (Pin_4), J4.4 (Pin_4)
- net DRAIN_GREEN: now also J3.2 (Pin_2), J4.2 (Pin_2); no longer J3.3 (Pin_3), J4.3 (Pin_3)
- net DRAIN_RED: now also J3.1 (Pin_1), J4.1 (Pin_1); no longer J3.2 (Pin_2), J4.2 (Pin_2)
- net GND: now also R12.1
Other:
- moved on the sheet: R1, R3, R5
Changed lines of the file:
@@
 L power:+12V #PWR010
 U 1 1 5DED5D2A
-P 9700 4300
-F 0 "#PWR010" H 9700 4150 50  0001 C CNN
-F 1 "+12V" H 9715 4473 50  0000 C CNN
-F 2 "" H 9700 4300 50  0001 C CNN
-F 3 "" H 9700 4300 50  0001 C CNN
-	1    9700 4300
-	1    0    0    -1
+P 9700 4700
+F 0 "#PWR010" H 9700 4550 50  0001 C CNN
+F 1 "+12V" H 9715 4873 50  0000 C CNN
+F 2 "" H 9700 4700 50  0001 C CNN
+F 3 "" H 9700 4700 50  0001 C CNN
+	1    9700 4700
+	-1   0    0    1
 $EndComp
 Wire Wire Line
 	9900 4400 9700 4400
 Wire Wire Line
-	9700 4400 9700 4300
-Wire Wire Line
 	9900 4500 9700 4500
 Wire Wire Line
@@
 Wire Wire Line
 	9900 4700 9700 4700
+Text Label 9700 4400 2    50   ~ 0
+DRAIN_RED
 Text Label 9700 4500 2    50   ~ 0
-DRAIN_RED
+DRAIN_GREEN
 Text Label 9700 4600 2    50   ~ 0
-DRAIN_GREEN
-Text Label 9700 4700 2    50   ~ 0
 DRAIN_BLUE
 $Comp
@@
 L power:+12V #PWR09
 U 1 1 5DED755F
-P 9700 3400
-F 0 "#PWR09" H 9700 3250 50  0001 C CNN
-F 1 "+12V" H 9715 3573 50  0000 C CNN
-F 2 "" H 9700 3400 50  0001 C CNN
-F 3 "" H 9700 3400 50  0001 C CNN
-	1    9700 3400
-	1    0    0    -1
+P 9700 3850
+F 0 "#PWR09" H 9700 3700 50  0001 C CNN
+F 1 "+12V" H 9715 4023 50  0000 C CNN
+F 2 "" H 9700 3850 50  0001 C CNN
+F 3 "" H 9700 3850 50  0001 C CNN
+	1    9700 3850
+	-1   0    0    1
 $EndComp
 Wire Wire Line
 	9900 3550 9700 3550
 Wire Wire Line
-	9700 3550 9700 3400
-Wire Wire Line
 	9900 3650 9700 3650
 Wire Wire Line
@@
 Wire Wire Line
 	9900 3850 9700 3850
+Text Label 9700 3550 2    50   ~ 0
+DRAIN_RED
 Text Label 9700 3650 2    50   ~ 0
-DRAIN_RED
+DRAIN_GREEN
 Text Label 9700 3750 2    50   ~ 0
-DRAIN_GREEN
-Text Label 9700 3850 2    50   ~ 0
 DRAIN_BLUE
 $Comp
@@
 	7500 1800 7500 1600
 Wire Wire Line
-	7300 1500 7250 1500
-Wire Wire Line
 	6950 1500 6950 1250
 Wire Wire Line
@@
 Wire Wire Line
 	6950 1900 6950 1800
-$Comp
-L Diode:1N4148W D1
-U 1 1 5DEF6A71
-P 6650 1500
-F 0 "D1" H 6650 1717 50  0000 C CNN
-F 1 "1N4148W" H 6650 1626 50  0000 C CNN
-F 2 "Diode_SMD:D_SOD-123" H 6650 1325 50  0001 C CNN
-F 3 "https://www.vishay.com/docs/85748/1n4148w.pdf" H 6650 1500 50  0001 C CNN
-	1    6650 1500
-	1    0    0    -1
-$EndComp
-Wire Wire Line
-	6950 1500 6800 1500
-Wire Wire Line
-	6500 1500 6350 1500
-Wire Wire Line
-	6350 1500 6350 1050
 Wire Wire Line
 	6350 1050 6650 1050
-Connection ~ 6350 1500
 $Comp
 L Device:R_Small R1
 U 1 1 5DEFA2D9
-P 6050 1500
-F 0 "R1" V 5854 1500 50  0000 C CNN
-F 1 "1K" V 5945 1500 50  0000 C CNN
-F 2 "Resistor_SMD:R_0805_2012Metric_Pad1.15x1.40mm_HandSolder" H 6050 1500 50  0001 C CNN
-F 3 "~" H 6050 1500 50  0001 C CNN
-	1    6050 1500
+P 6250 1050
+F 0 "R1" V 6054 1050 50  0000 C CNN
+F 1 "1K" V 6145 1050 50  0000 C CNN
+F 2 "Resistor_SMD:R_0805_2012Metric_Pad1.15x1.40mm_HandSolder" H 6250 1050 50  0001 C CNN
+F 3 "~" H 6250 1050 50  0001 C CNN
+	1    6250 1050
 	0    1    1    0
 $EndComp
 Wire Wire Line
-	6150 1500 6350 1500
-Wire Wire Line
-	5950 1500 5850 1500
+	6150 1050 6050 1050
 $Comp
 L Transistor_BJT:BC807 Q3
@@
 	7500 3450 7500 3250
 Wire Wire Line
-	7300 3150 7250 3150
-Wire Wire Line
 	6950 3150 6950 2900
 Wire Wire Line
@@
 Wire Wire Line
 	6950 3550 6950 3450
-$Comp
-L Diode:1N4148W D2
-U 1 1 5DF0155E
-P 6650 3150
-F 0 "D2" H 6650 3367 50  0000 C CNN
-F 1 "1N4148W" H 6650 3276 50  0000 C CNN
-F 2 "Diode_SMD:D_SOD-123" H 6650 2975 50  0001 C CNN
-F 3 "https://www.vishay.com/docs/85748/1n4148w.pdf" H 6650 3150 50  0001 C CNN
-	1    6650 3150
-	1    0    0    -1
-$EndComp
-Wire Wire Line
-	6950 3150 6800 3150
-Wire Wire Line
-	6500 3150 6350 3150
-Wire Wire Line
-	6350 3150 6350 2700
 Wire Wire Line
 	6350 2700 6650 2700
-Connection ~ 6350 3150
 $Comp
 L Device:R_Small R3
 U 1 1 5DF01569
-P 6050 3150
-F 0 "R3" V 5854 3150 50  0000 C CNN
-F 1 "1K" V 5945 3150 50  0000 C CNN
-F 2 "Resistor_SMD:R_0805_2012Metric_Pad1.15x1.40mm_HandSolder" H 6050 3150 50  0001 C CNN
-F 3 "~" H 6050 3150 50  0001 C CNN
-	1    6050 3150
+P 6250 2700
+F 0 "R3" V 6054 2700 50  0000 C CNN
+F 1 "1K" V 6145 2700 50  0000 C CNN
+F 2 "Resistor_SMD:R_0805_2012Metric_Pad1.15x1.40mm_HandSolder" H 6250 2700 50  0001 C CNN
+F 3 "~" H 6250 2700 50  0001 C CNN
+	1    6250 2700
 	0    1    1    0
 $EndComp
-Wire Wire Line
-	6150 3150 6350 3150
-Wire Wire Line
-	5950 3150 5900 3150
 $Comp
 L Transistor_BJT:BC807 Q5
@@
 	7500 5200 7500 5000
 Wire Wire Line
-	7300 4900 7200 4900
-Wire Wire Line
 	6950 4900 6950 4650
 Wire Wire Line
@@
 	6950 5300 6950 5200
 $Comp
-L Diode:1N4148W D3
-U 1 1 5DF053C1
-P 6650 4900
-F 0 "D3" H 6650 5117 50  0000 C CNN
-F 1 "1N4148W" H 6650 5026 50  0000 C CNN
-F 2 "Diode_SMD:D_SOD-123" H 6650 4725 50  0001 C CNN
-F 3 "https://www.vishay.com/docs/85748/1n4148w.pdf" H 6650 4900 50  0001 C CNN
-	1    6650 4900
-	1    0    0    -1
-$EndComp
-Wire Wire Line
-	6950 4900 6800 4900
-Wire Wire Line
-	6500 4900 6350 4900
-Wire Wire Line
-	6350 4900 6350 4450
-Wire Wire Line
-	6350 4450 6650 4450
-Connection ~ 6350 4900
-$Comp
 L Device:R_Small R5
 U 1 1 5DF053CC
-P 6050 4900
-F 0 "R5" V 5854 4900 50  0000 C CNN
-F 1 "1K" V 5945 4900 50  0000 C CNN
-F 2 "Resistor_SMD:R_0805_2012Metric_Pad1.15x1.40mm_HandSolder" H 6050 4900 50  0001 C CNN
-F 3 "~" H 6050 4900 50  0001 C CNN
-	1    6050 4900
+P 6350 4450
+F 0 "R5" V 6154 4450 50  0000 C CNN
+F 1 "1K" V 6245 4450 50  0000 C CNN
+F 2 "Resistor_SMD:R_0805_2012Metric_Pad1.15x1.40mm_HandSolder" H 6350 4450 50  0001 C CNN
+F 3 "~" H 6350 4450 50  0001 C CNN
+	1    6350 4450
 	0    1    1    0
 $EndComp
 Wire Wire Line
-	6150 4900 6350 4900
-Wire Wire Line
-	5950 4900 5850 4900
+	6250 4450 6200 4450
 Text Label 7750 1050 0    50   ~ 0
 DRAIN_RED
@@
 Text Label 7750 4450 0    50   ~ 0
 DRAIN_BLUE
-Text Label 5850 1500 2    50   ~ 0
+Text Label 6050 1050 2    50   ~ 0
 SIG_RED
-Text Label 5850 3150 2    50   ~ 0
+Text Label 6050 2700 2    50   ~ 0
 SIG_GREEN
-Text Label 5850 4900 2    50   ~ 0
+Text Label 6200 4450 2    50   ~ 0
 SIG_BLUE
 $Comp
@@
 	1    0    0    -1
 $EndComp
-$Comp
-L Jumper:SolderJumper_2_Open JP1
-U 1 1 5DF95CB7
-P 6300 2200
-F 0 "JP1" H 6300 2405 50  0000 C CNN
-F 1 "Red" H 6300 2314 50  0000 C CNN
-F 2 "Jumper:SolderJumper-2_P1.3mm_Open_RoundedPad1.0x1.5mm" H 6300 2200 50  0001 C CNN
-F 3 "~" H 6300 2200 50  0001 C CNN
-	1    6300 2200
-	1    0    0    -1
-$EndComp
-Wire Wire Line
-	6150 2200 5850 2200
-Wire Wire Line
-	5850 2200 5850 1500
-Wire Wire Line
-	7250 1500 7250 2200
-Wire Wire Line
-	7250 2200 6450 2200
-Connection ~ 7250 1500
-Wire Wire Line
-	7250 1500 6950 1500
-$Comp
-L Jumper:SolderJumper_2_Open JP2
-U 1 1 5DFA0EDD
-P 6350 3800
-F 0 "JP2" H 6350 4005 50  0000 C CNN
-F 1 "Green" H 6350 3914 50  0000 C CNN
-F 2 "Jumper:SolderJumper-2_P1.3mm_Open_RoundedPad1.0x1.5mm" H 6350 3800 50  0001 C CNN
-F 3 "~" H 6350 3800 50  0001 C CNN
-	1    6350 3800
-	1    0    0    -1
-$EndComp
-Wire Wire Line
-	7250 3150 7250 3800
-Wire Wire Line
-	7250 3800 6500 3800
-Connection ~ 7250 3150
-Wire Wire Line
-	7250 3150 6950 3150
-Wire Wire Line
-	5900 3150 5900 3800
-Wire Wire Line
-	5900 3800 6200 3800
-Connection ~ 5900 3150
-Wire Wire Line
-	5900 3150 5850 3150
-$Comp
-L Jumper:SolderJumper_2_Open JP3
-U 1 1 5DFAA680
-P 6450 5650
-F 0 "JP3" H 6450 5855 50  0000 C CNN
-F 1 "Blue" H 6450 5764 50  0000 C CNN
-F 2 "Jumper:SolderJumper-2_P1.3mm_Open_RoundedPad1.0x1.5mm" H 6450 5650 50  0001 C CNN
-F 3 "~" H 6450 5650 50  0001 C CNN
-	1    6450 5650
-	1    0    0    -1
-$EndComp
-Wire Wire Line
-	7200 4900 7200 5650
-Wire Wire Line
-	7200 5650 6600 5650
-Connection ~ 7200 4900
-Wire Wire Line
-	7200 4900 6950 4900
-Wire Wire Line
-	6300 5650 5850 5650
-Wire Wire Line
-	5850 5650 5850 4900
 Text Label 1700 1350 0    50   ~ 0
 BTN_RST
@@
 Text Label 3150 2200 0    50   ~ 0
 SIG_BLUE
+Wire Wire Line
+	6950 4900 7300 4900
+Wire Wire Line
+	6450 4450 6650 4450
+Wire Wire Line
+	6050 2700 6150 2700
+Wire Wire Line
+	6950 3150 7300 3150
+Wire Wire Line
+	6950 1500 7300 1500
+$Comp
+L Device:R_Small R12
+U 1 1 5DFA3EE6
+P 9200 5600
+F 0 "R12" H 9259 5646 50  0000 L CNN
+F 1 "100K" H 9259 5555 50  0000 L CNN
+F 2 "Resistor_SMD:R_0805_2012Metric_Pad1.15x1.40mm_HandSolder" H 9200 5600 50  0001 C CNN
+F 3 "~" H 9200 5600 50  0001 C CNN
+	1    9200 5600
+	1    0    0    1
+$EndComp
+$Comp
+L power:+12V #PWR0107
+U 1 1 5DFA4300
+P 9200 5400
+F 0 "#PWR0107" H 9200 5250 50  0001 C CNN
+F 1 "+12V" H 9215 5573 50  0000 C CNN
+F 2 "" H 9200 5400 50  0001 C CNN
+F 3 "" H 9200 5400 50  0001 C CNN
+	1    9200 5400
+	1    0    0    -1
+$EndComp
+Wire Wire Line
+	9200 5500 9200 5400
+$Comp
+L power:GND #PWR0108
+U 1 1 5DFA9DC4
+P 9200 5850
+F 0 "#PWR0108" H 9200 5600 50  0001 C CNN
+F 1 "GND" H 9205 5677 50  0000 C CNN
+F 2 "" H 9200 5850 50  0001 C CNN
+F 3 "" H 9200 5850 50  0001 C CNN
+	1    9200 5850
+	1    0    0    -1
+$EndComp
+Wire Wire Line
+	9200 5850 9200 5700
 $EndSCHEMATC

Commit message: finished board design
Parts:
- added Q7, Q8, Q9: BC817, Package_TO_SOT_SMD:SOT-23, symbol Transistor_BJT:BC817
- added R13, R14, R15: 1K, Resistor_SMD:R_0805_2012Metric_Pad1.15x1.40mm_HandSolder, symbol Device:R_Small
- added R16, R17, R18: 100R, Resistor_SMD:R_0805_2012Metric_Pad1.15x1.40mm_HandSolder, symbol Device:R_Small
- R2, R4, R6: value 100R -> 1K
Connections:
- net +12V: now also R13.2, R14.2, R15.2
- net GND: now also Q8.2 (E), Q9.2 (E)
- net at Q1.1 (B): now also Q8.3 (C), R14.1; no longer R1.1
- net at Q2.1 (G), R2.1: now also R16.1; no longer Q1.2 (E)
- net at R3.1: now also Q9.1 (B); no longer Q3.1 (B)
- net at Q4.1 (G), R4.1: now also R18.1; no longer Q3.2 (E)
- net at Q5.1 (B): now also Q7.3 (C), R13.1; no longer R5.1
- net at Q6.1 (G), R6.1: now also R17.1; no longer Q5.2 (E)
- new net: Q3.1 (B), Q9.3 (C), R15.1
- new net: Q1.2 (E), R16.2
- new net: Q8.1 (B), R1.1
- new net: Q3.2 (E), R18.2
- new net: Q5.2 (E), R17.2
- new net: Q7.1 (B), R5.1
Other:
- moved on the sheet: Q2, Q4, Q6, R1, R2, R3, R4, R5, R6

Commit message: Modified connectors and silkscreens. Added a diode to keep capacitor from charging during flashing. Added a second layer to mosfet connector traces and stiched them to help power dissipation.
Parts:
- removed J3: Conn_01x04, Connector_PinHeader_2.54mm:PinHeader_1x04_P2.54mm_Vertical, symbol Connector_Generic:Conn_01x04
- added D1: 1N4148, Diode_SMD:D_SOD-123, symbol Diode:1N4148
- J2: footprint Connector_PinHeader_2.54mm:PinHeader_1x06_P2.54mm_Vertical -> led_controller:Header_Programming
- J4: footprint TerminalBlock_RND:TerminalBlock_RND_205-00047_1x04_P5.00mm_Horizontal -> led_controller:connector_led
Connections:
- net +12V: now also D1.2 (A); no longer J2.1 (Pin_1), U1.3 (VI)
- net BTN_RST: now also J2.5 (Pin_5); no longer J2.2 (Pin_2)
- net FL_DTR: now also J2.4 (Pin_4); no longer J2.5 (Pin_5)
- net FL_TX: now also J2.2 (Pin_2); no longer J2.4 (Pin_4)
- new net +12L: D1.1 (K), J2.1 (Pin_1), U1.3 (VI)
Changed lines of the file:
@@
 F 0 "J4" H 10180 4492 50  0000 L CNN
 F 1 "Screw_Terminal_01x04" H 10180 4401 50  0000 L CNN
-F 2 "TerminalBlock_RND:TerminalBlock_RND_205-00047_1x04_P5.00mm_Horizontal" H 10100 4500 50  0001 C CNN
+F 2 "led_controller:connector_led" H 10100 4500 50  0001 C CNN
 F 3 "~" H 10100 4500 50  0001 C CNN
 	1    10100 4500
@@
 DRAIN_BLUE
 $Comp
-L Connector_Generic:Conn_01x04 J3
-U 1 1 5DED68AF
-P 10100 3650
-F 0 "J3" H 10180 3642 50  0000 L CNN
-F 1 "Conn_01x04" H 10180 3551 50  0000 L CNN
-F 2 "Connector_PinHeader_2.54mm:PinHeader_1x04_P2.54mm_Vertical" H 10100 3650 50  0001 C CNN
-F 3 "~" H 10100 3650 50  0001 C CNN
-	1    10100 3650
-	1    0    0    -1
-$EndComp
-$Comp
-L power:+12V #PWR09
-U 1 1 5DED755F
-P 9700 3850
-F 0 "#PWR09" H 9700 3700 50  0001 C CNN
-F 1 "+12V" H 9715 4023 50  0000 C CNN
-F 2 "" H 9700 3850 50  0001 C CNN
-F 3 "" H 9700 3850 50  0001 C CNN
-	1    9700 3850
-	-1   0    0    1
-$EndComp
-Wire Wire Line
-	9900 3550 9700 3550
-Wire Wire Line
-	9900 3650 9700 3650
-Wire Wire Line
-	9700 3750 9900 3750
-Wire Wire Line
-	9900 3850 9700 3850
-Text Label 9700 3550 2    50   ~ 0
-DRAIN_RED
-Text Label 9700 3650 2    50   ~ 0
-DRAIN_GREEN
-Text Label 9700 3750 2    50   ~ 0
-DRAIN_BLUE
-$Comp
 L Connector_Generic:Conn_01x06 J2
 U 1 1 5DED9194
@@
 F 0 "J2" H 10180 2492 50  0000 L CNN
 F 1 "Conn_01x06" H 10180 2401 50  0000 L CNN
-F 2 "Connector_PinHeader_2.54mm:PinHeader_1x06_P2.54mm_Vertical" H 10100 2500 50  0001 C CNN
+F 2 "led_controller:Header_Programming" H 10100 2500 50  0001 C CNN
 F 3 "~" H 10100 2500 50  0001 C CNN
 	1    10100 2500
-	1    0    0    -1
-$EndComp
-$Comp
-L power:+12V #PWR07
-U 1 1 5DED9DA1
-P 9700 2150
-F 0 "#PWR07" H 9700 2000 50  0001 C CNN
-F 1 "+12V" H 9715 2323 50  0000 C CNN
-F 2 "" H 9700 2150 50  0001 C CNN
-F 3 "" H 9700 2150 50  0001 C CNN
-	1    9700 2150
 	1    0    0    -1
 $EndComp
@@
 	9700 2800 9700 2950
 Wire Wire Line
-	9900 2400 9700 2400
-Wire Wire Line
-	9900 2500 9700 2500
-Wire Wire Line
-	9900 2600 9700 2600
-Wire Wire Line
-	9900 2700 9700 2700
-Text Label 9700 2400 2    50   ~ 0
+	9900 2400 9800 2400
+Wire Wire Line
+	9900 2500 9800 2500
+Wire Wire Line
+	9900 2600 9800 2600
+Wire Wire Line
+	9900 2700 9800 2700
+Text Label 9800 2700 2    50   ~ 0
 FL_RST
-Text Label 9700 2500 2    50   ~ 0
+Text Label 9800 2500 2    50   ~ 0
 FL_RX
-Text Label 9700 2600 2    50   ~ 0
+Text Label 9800 2400 2    50   ~ 0
 FL_TX
-Text Label 9700 2700 2    50   ~ 0
+Text Label 9800 2600 2    50   ~ 0
 FL_DTR
 $Comp
@@
 	1    0    0    -1
 $EndComp
-$Comp
-L power:+12V #PWR016
-U 1 1 5DF54C88
-P 1200 4600
-F 0 "#PWR016" H 1200 4450 50  0001 C CNN
-F 1 "+12V" H 1215 4773 50  0000 C CNN
-F 2 "" H 1200 4600 50  0001 C CNN
-F 3 "" H 1200 4600 50  0001 C CNN
-	1    1200 4600
-	1    0    0    -1
-$EndComp
 Wire Wire Line
 	1450 4700 1200 4700
@@
 	7250 4900 7650 4900
 Connection ~ 7650 4900
+$Comp
+L Diode:1N4148 D1
+U 1 1 5DF28498
+P 6900 5850
+F 0 "D1" H 6900 5634 50  0000 C CNN
+F 1 "1N4148" H 6900 5725 50  0000 C CNN
+F 2 "Diode_SMD:D_SOD-123" H 6900 5675 50  0001 C CNN
+F 3 "https://assets.nexperia.com/documents/data-sheet/1N4148_1N4448.pdf" H 6900 5850 50  0001 C CNN
+	1    6900 5850
+	1    0    0    1
+$EndComp
+$Comp
+L power:+12L #PWR0109
+U 1 1 5DF297EC
+P 6600 5750
+F 0 "#PWR0109" H 6600 5600 50  0001 C CNN
+F 1 "+12L" H 6615 5923 50  0000 C CNN
+F 2 "" H 6600 5750 50  0001 C CNN
+F 3 "" H 6600 5750 50  0001 C CNN
+	1    6600 5750
+	1    0    0    -1
+$EndComp
+$Comp
+L power:+12V #PWR0110
+U 1 1 5DF2F8C4
+P 7200 5750
+F 0 "#PWR0110" H 7200 5600 50  0001 C CNN
+F 1 "+12V" H 7215 5923 50  0000 C CNN
+F 2 "" H 7200 5750 50  0001 C CNN
+F 3 "" H 7200 5750 50  0001 C CNN
+	1    7200 5750
+	1    0    0    -1
+$EndComp
+Wire Wire Line
+	7200 5700 7200 5750
+Wire Wire Line
+	7200 5850 7050 5850
+Wire Wire Line
+	6600 5750 6600 5850
+Wire Wire Line
+	6600 5850 6750 5850
+Connection ~ 7200 5750
+Wire Wire Line
+	7200 5750 7200 5850
+$Comp
+L power:+12L #PWR0111
+U 1 1 5DF42305
+P 1200 4600
+F 0 "#PWR0111" H 1200 4450 50  0001 C CNN
+F 1 "+12L" H 1215 4773 50  0000 C CNN
+F 2 "" H 1200 4600 50  0001 C CNN
+F 3 "" H 1200 4600 50  0001 C CNN
+	1    1200 4600
+	1    0    0    -1
+$EndComp
+$Comp
+L power:+12L #PWR0112
+U 1 1 5DF449D2
+P 9700 2150
+F 0 "#PWR0112" H 9700 2000 50  0001 C CNN
+F 1 "+12L" H 9715 2323 50  0000 C CNN
+F 2 "" H 9700 2150 50  0001 C CNN
+F 3 "" H 9700 2150 50  0001 C CNN
+	1    9700 2150
+	1    0    0    -1
+$EndComp
 $EndSCHEMATC
